File: pcb_fsmc_ice40/pcb_fsmc_ice40.kicad_pcb (KiCad board)
At the start: 2 copper layers, 76.2 x 48 mm, 44 parts, among them P1 SD_CARD, P2 CONN_02X20, P5 CONN_02X12, P7 KNUSB, SW1 SWITCH_INV, U1 STM32F40X_LQFP144, X1 CRYSTAL

Commit message: Silk screen addition.
Other:
- board text added: "STM32F405 / FSMC module for ICE40-HX8K breakout board rev1 knielsen@knielsen-hq.org"
Changed lines of the file:
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@@
     (area 99.924999 83.924999 176.275001 132.075001)
     (thickness 1.6)
-    (drawings 44)
+    (drawings 45)
     (tracks 880)
     (zones 0)
@@
     )
   )
+  (gr_text "STM32F405 / FSMC\nmodule for ICE40-HX8K\nbreakout board   rev1\n\nknielsen@knielsen-hq.org" (at 145.1 120) (layer F.SilkS)
+    (effects (font (size 1.5 1.5) (thickness 0.3)) (justify left))
+  )
   (gr_text RESET (at 113.9 92.1) (layer B.SilkS)
